Commit message: Tang deadband len 4.0N va xoay he toa do luc

File: src/hc10dtp_moveit_config/config/motoman_hc10dtp.ros2_control.xacro (robot description, xacro)
@@ -1,5 +1,5 @@
 <?xml version="1.0"?>
 <robot xmlns:xacro="http://www.ros.org/wiki/xacro">
-    <xacro:macro name="motoman_hc10dtp_ros2_control" params="name initial_positions_file use_fake_hardware:=false robot_ip:=192.168.1.33 controller_port:=50240">
+    <xacro:macro name="motoman_hc10dtp_ros2_control" params="name initial_positions_file use_fake_hardware:=false robot_ip:=192.168.1.53 controller_port:=50240">
         <xacro:property name="initial_positions" value="${xacro.load_yaml(initial_positions_file)['initial_positions']}"/>
         <ros2_control name="${name}" type="system">

File: src/hc10dtp_moveit_config/config/motoman_hc10dtp.urdf.xacro (robot description, xacro)
@@ -3,5 +3,5 @@
     <xacro:arg name="initial_positions_file" default="initial_positions.yaml" />
     <xacro:arg name="use_fake_hardware"       default="false" />
-    <xacro:arg name="robot_ip"                default="192.168.1.33" />
+    <xacro:arg name="robot_ip"                default="192.168.1.53" />
     <xacro:arg name="controller_port"         default="50240" />
     <!-- Import HC10DTP URDF -->

File: src/motoman_hc10dtp_support/urdf/hc10dtp_b00_macro_custom.xacro (robot description, xacro)
@@ -156,4 +156,11 @@
       <child link="${prefix}tool0"/>
     </joint>
+    <!-- Axia80 Force/Torque Sensor Frame -->
+    <link name="${prefix}axia_sensor_link"/>
+    <joint name="${prefix}tool0-axia_sensor" type="fixed">
+      <origin xyz="0 0 0" rpy="0 0 ${radians(-152.7)}"/>
+      <parent link="${prefix}tool0"/>
+      <child link="${prefix}axia_sensor_link"/>
+    </joint>
   </xacro:macro>
 </robot>
