Commit message: Chay thanh cong che do x_ref = Home voi robot that + train GRU

File: src/motoman_hc10dtp_support/urdf/hc10dtp_b00_macro_custom.xacro (robot description, xacro)
@@ -159,5 +159,5 @@
     <link name="${prefix}axia_sensor_link"/>
     <joint name="${prefix}tool0-axia_sensor" type="fixed">
-      <origin xyz="0 0 0" rpy="0 0 ${radians(-152.7)}"/>
+      <origin xyz="0 0 0" rpy="0 0 ${radians(61.2)}"/>
       <parent link="${prefix}tool0"/>
       <child link="${prefix}axia_sensor_link"/>
